File: MotorDriver_TMC2660.sch (KiCad schematic (older format))
At the start: 17 parts, among them U4 TMC2660

Commit message: Added clock line for the motor drivers.
Parts:
- added JP?: Clk Disable, symbol Jumper:SolderJumper_2_Open
Connections:
- net GND: now also JP?.2 (B); no longer U4.21 (CLK)
- new net CLOCK: JP?.1 (A), U4.21 (CLK)
Changed lines of the file:
@@
 AR Path="/5AC337B6/5ACE1C6D/5ACC0B66/5AC338BF" Ref="U7"  Part="1"
 AR Path="/5AC337B6/5AD9F95A/5AD4B0F5/5AC338BF" Ref="U8"  Part="1"
-F 0 "U7" H 4875 2520 60  0000 C CNN
+F 0 "U5" H 4875 2520 60  0000 C CNN
 F 1 "TMC2660" H 4875 2414 60  0000 C CNN
 F 2 "PrntrBoardV1:TMC2660" H 4900 3600 60  0001 C CNN
@@
 AR Path="/5AC337B6/5ACE1C6D/5ACC0B66/5AC33A94" Ref="C46"  Part="1"
 AR Path="/5AC337B6/5AD9F95A/5AD4B0F5/5AC33A94" Ref="C59"  Part="1"
-F 0 "C46" H 4650 1800 50  0000 L CNN
+F 0 "C20" H 4650 1800 50  0000 L CNN
 F 1 "0.1uF 50V" H 4350 1550 50  0000 L CNN
 F 2 "Capacitor_SMD:C_0603_1608Metric" H 4638 1550 50  0001 C CNN
@@
 AR Path="/5AC337B6/5ACE1C6D/5ACC0B66/5AC33B3C" Ref="C44"  Part="1"
 AR Path="/5AC337B6/5AD9F95A/5AD4B0F5/5AC33B3C" Ref="C57"  Part="1"
-F 0 "C44" H 3050 1750 50  0000 L CNN
+F 0 "C18" H 3050 1750 50  0000 L CNN
 F 1 "10uF 50V" H 2850 1650 50  0000 L CNN
 F 2 "Capacitor_SMD:C_1206_3216Metric" H 3338 1550 50  0001 C CNN
@@
 AR Path="/5AC337B6/5ACE1C6D/5ACC0B66/5AC33B85" Ref="C47"  Part="1"
 AR Path="/5AC337B6/5AD9F95A/5AD4B0F5/5AC33B85" Ref="C60"  Part="1"
-F 0 "C47" V 5098 2100 50  0000 C CNN
+F 0 "C21" V 5098 2100 50  0000 C CNN
 F 1 "0.47uF" V 5189 2100 50  0000 C CNN
 F 2 "Capacitor_SMD:C_0603_1608Metric" H 5388 1950 50  0001 C CNN
@@
 AR Path="/5AC337B6/5ACE1C6D/5ACC0B66/5AC33C56" Ref="C48"  Part="1"
 AR Path="/5AC337B6/5AD9F95A/5AD4B0F5/5AC33C56" Ref="C61"  Part="1"
-F 0 "C48" H 5765 1896 50  0000 L CNN
+F 0 "C22" H 5765 1896 50  0000 L CNN
 F 1 "0.1uF" H 5765 1805 50  0000 L CNN
 F 2 "Capacitor_SMD:C_0603_1608Metric" H 5688 1700 50  0001 C CNN
@@
 AR Path="/5AC337B6/5ACE1C6D/5ACC0B66/5AC33CA1" Ref="C50"  Part="1"
 AR Path="/5AC337B6/5AD9F95A/5AD4B0F5/5AC33CA1" Ref="C63"  Part="1"
-F 0 "C50" V 6300 2600 50  0000 C CNN
+F 0 "C24" V 6300 2600 50  0000 C CNN
 F 1 "1000pF >50V" V 6400 2700 50  0000 C CNN
 F 2 "Capacitor_SMD:C_0603_1608Metric" H 6238 2600 50  0001 C CNN
@@
 AR Path="/5AC337B6/5ACE1C6D/5ACC0B66/5AC33D6E" Ref="C51"  Part="1"
 AR Path="/5AC337B6/5AD9F95A/5AD4B0F5/5AC33D6E" Ref="C64"  Part="1"
-F 0 "C51" V 6300 3000 50  0000 C CNN
+F 0 "C25" V 6300 3000 50  0000 C CNN
 F 1 "1000pF >50V" V 6400 3100 50  0000 C CNN
 F 2 "Capacitor_SMD:C_0603_1608Metric" H 6238 3000 50  0001 C CNN
@@
 AR Path="/5AC337B6/5ACE1C6D/5ACC0B66/5AC33DC1" Ref="C52"  Part="1"
 AR Path="/5AC337B6/5AD9F95A/5AD4B0F5/5AC33DC1" Ref="C65"  Part="1"
-F 0 "C52" V 6300 3700 50  0000 C CNN
+F 0 "C26" V 6300 3700 50  0000 C CNN
 F 1 "1000pF >50V" V 6400 3850 50  0000 C CNN
 F 2 "Capacitor_SMD:C_0603_1608Metric" H 6238 3700 50  0001 C CNN
@@
 AR Path="/5AC337B6/5ACE1C6D/5ACC0B66/5AC33E6E" Ref="C53"  Part="1"
 AR Path="/5AC337B6/5AD9F95A/5AD4B0F5/5AC33E6E" Ref="C66"  Part="1"
-F 0 "C53" V 6300 4150 50  0000 C CNN
+F 0 "C27" V 6300 4150 50  0000 C CNN
 F 1 "1000pF >50V" V 6400 4250 50  0000 C CNN
 F 2 "Capacitor_SMD:C_0603_1608Metric" H 6238 4100 50  0001 C CNN
@@
 AR Path="/5AC337B6/5ACE1C6D/5ACC0B66/5AC33EDF" Ref="C54"  Part="1"
 AR Path="/5AC337B6/5AD9F95A/5AD4B0F5/5AC33EDF" Ref="C67"  Part="1"
-F 0 "C54" H 7300 4550 50  0000 L CNN
+F 0 "C28" H 7300 4550 50  0000 L CNN
 F 1 "0.01uF X7R 10% 50V" H 7550 4550 50  0000 L CNN
 F 2 "Capacitor_SMD:C_0603_1608Metric" H 7238 4400 50  0001 C CNN
@@
 AR Path="/5AC337B6/5ACE1C6D/5ACC0B66/5AC33F7D" Ref="C49"  Part="1"
 AR Path="/5AC337B6/5AD9F95A/5AD4B0F5/5AC33F7D" Ref="C62"  Part="1"
-F 0 "C49" H 5650 5100 50  0000 L CNN
+F 0 "C23" H 5650 5100 50  0000 L CNN
 F 1 "0.01uF X7R 10% 50V" H 4950 5000 50  0000 L CNN
 F 2 "Capacitor_SMD:C_0603_1608Metric" H 5938 4900 50  0001 C CNN
@@
 AR Path="/5AC337B6/5ACE1C6D/5ACC0B66/5AC34593" Ref="#PWR049"  Part="1"
 AR Path="/5AC337B6/5AD9F95A/5AD4B0F5/5AC34593" Ref="#PWR059"  Part="1"
-F 0 "#PWR049" H 5650 1950 50  0001 C CNN
+F 0 "#PWR027" H 5650 1950 50  0001 C CNN
 F 1 "GND" H 5655 2027 50  0000 C CNN
 F 2 "" H 5650 2200 50  0001 C CNN
@@
 AR Path="/5AC337B6/5ACE1C6D/5ACC0B66/5AC345D6" Ref="#PWR048"  Part="1"
 AR Path="/5AC337B6/5AD9F95A/5AD4B0F5/5AC345D6" Ref="#PWR058"  Part="1"
-F 0 "#PWR048" H 3300 1800 50  0001 C CNN
+F 0 "#PWR026" H 3300 1800 50  0001 C CNN
 F 1 "GND" H 3305 1877 50  0000 C CNN
 F 2 "" H 3300 2050 50  0001 C CNN
@@
 AR Path="/5AC337B6/5ACE1C6D/5ACC0B66/5AC34619" Ref="#PWR050"  Part="1"
 AR Path="/5AC337B6/5AD9F95A/5AD4B0F5/5AC34619" Ref="#PWR060"  Part="1"
-F 0 "#PWR050" H 6450 2500 50  0001 C CNN
+F 0 "#PWR028" H 6450 2500 50  0001 C CNN
 F 1 "GND" H 6550 2750 50  0000 C CNN
 F 2 "" H 6450 2750 50  0001 C CNN
@@
 AR Path="/5AC337B6/5ACE1C6D/5ACC0B66/5AC3465C" Ref="#PWR051"  Part="1"
 AR Path="/5AC337B6/5AD9F95A/5AD4B0F5/5AC3465C" Ref="#PWR061"  Part="1"
-F 0 "#PWR051" H 6450 2900 50  0001 C CNN
+F 0 "#PWR029" H 6450 2900 50  0001 C CNN
 F 1 "GND" H 6550 3050 50  0000 C CNN
 F 2 "" H 6450 3150 50  0001 C CNN
@@
 AR Path="/5AC337B6/5ACE1C6D/5ACC0B66/5AC3469F" Ref="#PWR052"  Part="1"
 AR Path="/5AC337B6/5AD9F95A/5AD4B0F5/5AC3469F" Ref="#PWR062"  Part="1"
-F 0 "#PWR052" H 6450 3600 50  0001 C CNN
+F 0 "#PWR030" H 6450 3600 50  0001 C CNN
 F 1 "GND" H 6550 3850 50  0000 C CNN
 F 2 "" H 6450 3850 50  0001 C CNN
@@
 AR Path="/5AC337B6/5ACE1C6D/5ACC0B66/5AC346E2" Ref="#PWR053"  Part="1"
 AR Path="/5AC337B6/5AD9F95A/5AD4B0F5/5AC346E2" Ref="#PWR063"  Part="1"
-F 0 "#PWR053" H 6450 4000 50  0001 C CNN
+F 0 "#PWR031" H 6450 4000 50  0001 C CNN
 F 1 "GND" H 6550 4250 50  0000 C CNN
 F 2 "" H 6450 4250 50  0001 C CNN
@@
 AR Path="/5AC337B6/5ACE1C6D/5ACC0B66/5AC34725" Ref="#PWR047"  Part="1"
 AR Path="/5AC337B6/5AD9F95A/5AD4B0F5/5AC34725" Ref="#PWR057"  Part="1"
-F 0 "#PWR047" H 2950 6050 50  0001 C CNN
+F 0 "#PWR025" H 2950 6050 50  0001 C CNN
 F 1 "GND" H 2955 6127 50  0000 C CNN
 F 2 "" H 2950 6300 50  0001 C CNN
@@
 AR Path="/5AC337B6/5ACE1C6D/5ACC0B66/5AC3912E" Ref="R28"  Part="1"
 AR Path="/5AC337B6/5AD9F95A/5AD4B0F5/5AC3912E" Ref="R36"  Part="1"
-F 0 "R28" H 6050 4950 50  0000 L CNN
+F 0 "R12" H 6050 4950 50  0000 L CNN
 F 1 "22R" H 6050 4850 50  0000 L CNN
 F 2 "Resistor_SMD:R_0603_1608Metric" V 6180 4900 50  0001 C CNN
@@
 AR Path="/5AC337B6/5ACE1C6D/5ACC0B66/5AC391BE" Ref="R29"  Part="1"
 AR Path="/5AC337B6/5AD9F95A/5AD4B0F5/5AC391BE" Ref="R37"  Part="1"
-F 0 "R29" H 6320 5396 50  0000 L CNN
+F 0 "R13" H 6320 5396 50  0000 L CNN
 F 1 "0R051" H 6320 5305 50  0000 L CNN
 F 2 "Resistor_SMD:R_1206_3216Metric" V 6180 5350 50  0001 C CNN
@@
 AR Path="/5AC337B6/5ACE1C6D/5ACC0B66/5AC3921D" Ref="R30"  Part="1"
 AR Path="/5AC337B6/5AD9F95A/5AD4B0F5/5AC3921D" Ref="R38"  Part="1"
-F 0 "R30" H 7300 3900 50  0000 L CNN
+F 0 "R14" H 7300 3900 50  0000 L CNN
 F 1 "22R" H 7300 3800 50  0000 L CNN
 F 2 "Resistor_SMD:R_0603_1608Metric" V 7430 3850 50  0001 C CNN
@@
 AR Path="/5AC337B6/5ACE1C6D/5ACC0B66/5AC392A1" Ref="R31"  Part="1"
 AR Path="/5AC337B6/5AD9F95A/5AD4B0F5/5AC392A1" Ref="R39"  Part="1"
-F 0 "R31" H 7570 5196 50  0000 L CNN
+F 0 "R15" H 7570 5196 50  0000 L CNN
 F 1 "0R051" H 7570 5105 50  0000 L CNN
 F 2 "Resistor_SMD:R_1206_3216Metric" V 7430 5150 50  0001 C CNN
@@
 	3800 4450 3800 4550
 Wire Wire Line
-	3800 6000 3700 6000
-Wire Wire Line
 	4000 4550 3800 4550
 Connection ~ 3800 4550
@@
 	3800 4300 3800 4450
 Connection ~ 3800 4450
-Wire Wire Line
-	4000 3950 3700 3950
-Wire Wire Line
-	3700 3950 3700 6000
-Connection ~ 3700 6000
 Wire Wire Line
 	7500 3700 7500 3550
@@
 AR Path="/5AC337B6/5ACE1C6D/5ACC0B66/5AC55FA7" Ref="C45"  Part="1"
 AR Path="/5AC337B6/5AD9F95A/5AD4B0F5/5AC55FA7" Ref="C58"  Part="1"
-F 0 "C45" H 3700 1900 50  0000 L CNN
+F 0 "C19" H 3700 1900 50  0000 L CNN
 F 1 "100uF 35V" H 3700 1800 50  0000 L CNN
 F 2 "Capacitor_SMD:CP_Elec_6.3x7.7" H 3650 1700 50  0001 C CNN
@@
 	2950 6300 2950 6000
 Wire Wire Line
-	2950 6000 3700 6000
-Wire Wire Line
 	6350 3150 6450 3150
 $Comp
@@
 AR Path="/5AC337B6/5ACE1C6D/5ACC0B66/5ACA36B2" Ref="C76"  Part="1"
 AR Path="/5AC337B6/5AD9F95A/5AD4B0F5/5ACA36B2" Ref="C77"  Part="1"
-F 0 "C76" H 2715 1746 50  0000 L CNN
+F 0 "C74" H 2715 1746 50  0000 L CNN
 F 1 "10uF 50V" H 2650 1550 50  0000 L CNN
 F 2 "Capacitor_SMD:C_1206_3216Metric" H 2638 1550 50  0001 C CNN
@@
 Wire Wire Line
 	2600 2000 3300 2000
+Wire Wire Line
+	2950 6000 3600 6000
+$Comp
+L Jumper:SolderJumper_2_Open JP?
+U 1 1 5AF10E97
+P 3600 5050
+F 0 "JP?" V 3550 4850 50  0000 L CNN
+F 1 "Clk Disable" V 3650 4550 50  0000 L CNN
+F 2 "" H 3600 5050 50  0001 C CNN
+F 3 "~" H 3600 5050 50  0001 C CNN
+	1    3600 5050
+	0    1    1    0
+$EndComp
+Wire Wire Line
+	3600 5200 3600 6000
+Connection ~ 3600 6000
+Wire Wire Line
+	3600 6000 3800 6000
+Wire Wire Line
+	3600 4900 3600 3950
+Wire Wire Line
+	3600 3950 4000 3950
+Text HLabel 3250 3950 0    50   Input ~ 0
+CLOCK
+Wire Wire Line
+	3250 3950 3600 3950
+Connection ~ 3600 3950
 $EndSCHEMATC
