File: PrntrBoardV1.kicad_pcb (KiCad board)
At the start: 4 copper layers, 100 x 100.2 mm, 203 parts, among them J1 EXT 5V, J10 Probe, J11 Extruder Heater, J12 Stepper, J13 Thermistor, J14 Max, J15 Min, J16 Max, J17 Min, J18 Max, J19 Min, J2 Bed Heater, J20 Stepper, J21 Stepper, J22 Stepper, J23 Stepper, J24 Probe, J25 Extruder Heater, J26 Stepper, J27 Thermistor, J28 Thermistor, J29 12-24V, J3 Z Probe, J4 E0 Cool, J5 E0 Part, J6 E1 Cool, J7 E1 Part, J8 Always On Fan 1, J9 Always On Fan 2, U1 4078, U11 NUCLEO-64, U2 74HCT02, U3 74LVC125, U4 TMC2660, U5 TMC2660, U6 TMC2660, U7 TMC2660, U8 TMC2660

Commit message: All routed again. Clock jumpers on the bottom side.
Parts:
- added J30: Ext Clock, Connector_PinHeader_2.54mm:PinHeader_1x02_P2.54mm_Vertical, F.Cu at (114.6, 65.4)
- added JP2: Motor Clock Select, Jumper:SolderJumper-3_P1.3mm_Bridged2Bar12_Pad1.0x1.5mm, B.Cu at (108.6, 82.2)
- added JP3: Clk Disable, Jumper:SolderJumper-2_P1.3mm_Open_Pad1.0x1.5mm, B.Cu at (128.3, 111.8)
- added JP4: Clk Disable, Jumper:SolderJumper-2_P1.3mm_Open_Pad1.0x1.5mm, B.Cu at (128.2, 88.3)
- added JP5: Clk Disable, Jumper:SolderJumper-2_P1.3mm_Open_Pad1.0x1.5mm, B.Cu at (123.3, 63.1)
- added JP6: Clk Disable, Jumper:SolderJumper-2_P1.3mm_Open_Pad1.0x1.5mm, B.Cu at (71.9, 50.0)
- added JP7: Clk Disable, Jumper:SolderJumper-2_P1.3mm_Open_Pad1.0x1.5mm, B.Cu at (71.0, 27.7)
Connections:
- U4 pad 21: GND -> /MOT_CLOCK
- U5 pad 21: GND -> /MOT_CLOCK
- U6 pad 21: GND -> /MOT_CLOCK
- U7 pad 21: GND -> /MOT_CLOCK
- U8 pad 21: GND -> /MOT_CLOCK
Routing:
- net /MOT_CLOCK: track 0.00 -> 181.7 mm, vias 0 -> 6
- net Net-(J30-Pad2): track 0.00 -> 15.4 mm
- net Net-(JP2-Pad1): track 0.00 -> 11.9 mm
- net GND: track 189.5 -> 187.2 mm, vias 209 -> 210
- net /MotorControl/E0/~ENABLE: track 152.3 -> 151.2 mm

Commit message: Add motorl clock jumper labels.
Other:
- board text added: "Disable Mot Clk"
- board text added: "Ext Motor Clock"
- board text added: "Motor Clk Select (ext int)"
Changed lines of the file:
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@@
   (general
     (thickness 1.6)
-    (drawings 32)
+    (drawings 39)
     (tracks 3143)
     (zones 0)
@@
     )
   )
+  (gr_text "Motor Clk\nSelect\n(ext   int)" (at 108.4072 87.6554 90) (layer B.SilkS)
+    (effects (font (size 0.8 0.8) (thickness 0.1)) (justify mirror))
+  )
+  (gr_text "Disable\nMot Clk" (at 128.016 114.4778) (layer B.SilkS)
+    (effects (font (size 0.8 0.8) (thickness 0.1)) (justify mirror))
+  )
+  (gr_text "Disable\nMot Clk" (at 127.889 92.4814) (layer B.SilkS)
+    (effects (font (size 0.8 0.8) (thickness 0.1)) (justify mirror))
+  )
+  (gr_text "Disable\nMot Clk" (at 120.8532 66.0908) (layer B.SilkS)
+    (effects (font (size 0.8 0.8) (thickness 0.1)) (justify mirror))
+  )
+  (gr_text "Disable\nMot Clk" (at 75.7174 26.7208) (layer B.SilkS)
+    (effects (font (size 0.8 0.8) (thickness 0.1)) (justify mirror))
+  )
+  (gr_text "Disable\nMot Clk" (at 76.2254 49.5808) (layer B.SilkS)
+    (effects (font (size 0.8 0.8) (thickness 0.1)) (justify mirror))
+  )
+  (gr_text "Ext\nMotor\nClock" (at 109.093 65.3796) (layer F.SilkS)
+    (effects (font (size 1.5 1.5) (thickness 0.3)))
+  )
   (gr_text "NUCLEO-F446RE\nSTM32 ARM M4" (at 100.076 75.946) (layer B.SilkS)
