File: PrntrBoardV1.kicad_pcb (KiCad board)
At the start: 4 copper layers, 99 x 99 mm, 229 parts, among them J1 EXT 5V, J10 Probe, J11 Extruder Heater, J12 Stepper, J13 Thermistor, J14 Max, J15 Min, J16 Max, J17 Min, J18 Max, J19 Min, J2 Bed Heater, J20 Stepper, J21 Stepper, J22 Stepper, J23 Stepper, J24 Probe, J25 Extruder Heater, J26 Stepper, J27 Thermistor, J28 Thermistor, J29 12-24V, J3 Z Probe, J30 LCD, J31 TC1, J32 TC2, J4 E0 Cool, J5 E0 Part, J6 E1 Cool, J7 E1 Part, J8 Always On Fan 1, J9 Always On Fan 2, U1 4078, U11 NUCLEO-64, U2 74HCT02, U3 74LVC125, U4 TMC2660, U5 TMC2660, U6 TMC2660, U7 TMC2660, U8 TMC2660, X1 16MHz

Commit message: Rename some somponents to suite PNP process.
Parts:
- C11, C12, C13, C14, C26, C27, C28, C31, C40, C41, C44, C45, C54, C57, C58, C59, C73, C74, C75, C76: value 1000pF >50V -> 1000pF
- D10, D11, D2: value HEATER -> LED
Changed lines of the file:
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@@
-(kicad_pcb (version 20171130) (host pcbnew 5.0.0-rc2-unknown-68f6e3a~65~ubuntu18.04.1)
+(kicad_pcb (version 20171130) (host pcbnew 5.0.0-rc2-unknown-73a8d2a~65~ubuntu18.04.1)
   (general
     (thickness 1.6)
@@
       (drillshape 0)
       (scaleselection 1)
-      (outputdirectory Gerber/))
+      (outputdirectory "Gerber/"))
   )
   (net 0 "")
@@
       (effects (font (size 1 1) (thickness 0.15)))
     )
-    (fp_text value "1000pF >50V" (at 0 1.45 90) (layer F.Fab)
+    (fp_text value 1000pF (at 0 1.45 90) (layer F.Fab)
       (effects (font (size 1 1) (thickness 0.15)))
     )
@@
       (effects (font (size 1 1) (thickness 0.15)))
     )
-    (fp_text value "1000pF >50V" (at 0 1.45 180) (layer F.Fab)
+    (fp_text value 1000pF (at 0 1.45 180) (layer F.Fab)
       (effects (font (size 1 1) (thickness 0.15)))
     )
@@
       (effects (font (size 1 1) (thickness 0.15)))
     )
-    (fp_text value "1000pF >50V" (at 0 1.45 180) (layer F.Fab)
+    (fp_text value 1000pF (at 0 1.45 180) (layer F.Fab)
       (effects (font (size 1 1) (thickness 0.15)))
     )
@@
       (effects (font (size 1 1) (thickness 0.15)))
     )
-    (fp_text value "1000pF >50V" (at 0 1.45 180) (layer F.Fab)
+    (fp_text value 1000pF (at 0 1.45 180) (layer F.Fab)
       (effects (font (size 1 1) (thickness 0.15)))
     )
@@
       (effects (font (size 1 1) (thickness 0.15)))
     )
-    (fp_text value "1000pF >50V" (at 0 1.45 270) (layer F.Fab)
+    (fp_text value 1000pF (at 0 1.45 270) (layer F.Fab)
       (effects (font (size 1 1) (thickness 0.15)))
     )
@@
       (effects (font (size 1 1) (thickness 0.15)))
     )
-    (fp_text value "1000pF >50V" (at 0 1.45) (layer F.Fab)
+    (fp_text value 1000pF (at 0 1.45) (layer F.Fab)
       (effects (font (size 1 1) (thickness 0.15)))
     )
@@
       (effects (font (size 1 1) (thickness 0.15)))
     )
-    (fp_text value "1000pF >50V" (at 0 1.45) (layer F.Fab)
+    (fp_text value 1000pF (at 0 1.45) (layer F.Fab)
       (effects (font (size 1 1) (thickness 0.15)))
     )
@@
       (effects (font (size 1 1) (thickness 0.15)))
     )
-    (fp_text value "1000pF >50V" (at 0 1.45) (layer F.Fab)
+    (fp_text value 1000pF (at 0 1.45) (layer F.Fab)
       (effects (font (size 1 1) (thickness 0.15)))
     )
@@
       (effects (font (size 1 1) (thickness 0.15)))
     )
-    (fp_text value "1000pF >50V" (at 0 1.45 270) (layer F.Fab)
+    (fp_text value 1000pF (at 0 1.45 270) (layer F.Fab)
       (effects (font (size 1 1) (thickness 0.15)))
     )
@@
       (effects (font (size 1 1) (thickness 0.15)))
     )
-    (fp_text value "1000pF >50V" (at 0 1.45) (layer F.Fab)
+    (fp_text value 1000pF (at 0 1.45) (layer F.Fab)
       (effects (font (size 1 1) (thickness 0.15)))
     )
@@
       (effects (font (size 1 1) (thickness 0.15)))
     )
-    (fp_text value "1000pF >50V" (at 0 1.45) (layer F.Fab)
+    (fp_text value 1000pF (at 0 1.45) (layer F.Fab)
       (effects (font (size 1 1) (thickness 0.15)))
     )
@@
       (effects (font (size 1 1) (thickness 0.15)))
     )
-    (fp_text value "1000pF >50V" (at 0 1.45) (layer F.Fab)
+    (fp_text value 1000pF (at 0 1.45) (layer F.Fab)
       (effects (font (size 1 1) (thickness 0.15)))
     )
@@
       (effects (font (size 1 1) (thickness 0.15)))
     )
-    (fp_text value "1000pF >50V" (at 0 1.45 90) (layer F.Fab)
+    (fp_text value 1000pF (at 0 1.45 90) (layer F.Fab)
       (effects (font (size 1 1) (thickness 0.15)))
     )
@@
       (effects (font (size 1 1) (thickness 0.15)))
     )
-    (fp_text value "1000pF >50V" (at 0 1.45 90) (layer F.Fab)
+    (fp_text value 1000pF (at 0 1.45 90) (layer F.Fab)
       (effects (font (size 1 1) (thickness 0.15)))
     )
@@
       (effects (font (size 1 1) (thickness 0.15)))
     )
-    (fp_text value "1000pF >50V" (at 0 1.45 270) (layer F.Fab)
+    (fp_text value 1000pF (at 0 1.45 270) (layer F.Fab)
       (effects (font (size 1 1) (thickness 0.15)))
     )
@@
       (effects (font (size 1 1) (thickness 0.15)))
     )
-    (fp_text value "1000pF >50V" (at 0 1.45 270) (layer F.Fab)
+    (fp_text value 1000pF (at 0 1.45 270) (layer F.Fab)
       (effects (font (size 1 1) (thickness 0.15)))
     )
@@
       (effects (font (size 1 1) (thickness 0.15)))
     )
-    (fp_text value "1000pF >50V" (at 0 1.45) (layer F.Fab)
+    (fp_text value 1000pF (at 0 1.45) (layer F.Fab)
       (effects (font (size 1 1) (thickness 0.15)))
     )
@@
       (effects (font (size 1 1) (thickness 0.15)))
     )
-    (fp_text value "1000pF >50V" (at 0 1.45 90) (layer F.Fab)
+    (fp_text value 1000pF (at 0 1.45 90) (layer F.Fab)
       (effects (font (size 1 1) (thickness 0.15)))
     )
@@
       (effects (font (size 1 1) (thickness 0.15)))
     )
-    (fp_text value "1000pF >50V" (at 0 1.45 90) (layer F.Fab)
+    (fp_text value 1000pF (at 0 1.45 90) (layer F.Fab)
       (effects (font (size 1 1) (thickness 0.15)))
     )
@@
       (effects (font (size 1 1) (thickness 0.15)))
     )
-    (fp_text value "1000pF >50V" (at 0 1.45 90) (layer F.Fab)
+    (fp_text value 1000pF (at 0 1.45 90) (layer F.Fab)
       (effects (font (size 1 1) (thickness 0.15)))
     )
@@
       (effects (font (size 1 1) (thickness 0.15)))
     )
-    (fp_text value HEATER (at 0 1.45 270) (layer F.Fab)
+    (fp_text value LED (at 0 1.45 270) (layer F.Fab)
       (effects (font (size 1 1) (thickness 0.15)))
     )
@@
       (effects (font (size 1 1) (thickness 0.15)))
     )
-    (fp_text value HEATER (at 0 1.45 270) (layer F.Fab)
+    (fp_text value LED (at 0 1.45 270) (layer F.Fab)
       (effects (font (size 1 1) (thickness 0.15)))
     )
@@
       (effects (font (size 1 1) (thickness 0.15)))
     )
-    (fp_text value HEATER (at 0 1.45 270) (layer F.Fab)
+    (fp_text value LED (at 0 1.45 270) (layer F.Fab)
       (effects (font (size 1 1) (thickness 0.15)))
     )
