File: Extruder.sch (KiCad schematic (older format))
At the start: 2 parts, among them J10 Probe, J11 Extruder Heater

Commit message: Update connector components. Correct bad capacitor value.
Parts:
- J11: symbol Connector_Specialized:Screw_Terminal_01x02 -> Connector_Generic:Conn_01x02
Changed lines of the file:
@@
 $Descr A4 11693 8268
 encoding utf-8
-Sheet 25 34
+Sheet 3 34
 Title ""
 Date ""
@@
 AR Path="/5AC337B6/5ACBE919/5AD4BF35" Ref="J10"  Part="1"
 AR Path="/5AC337B6/5AD9F95A/5AD4BF35" Ref="J24"  Part="1"
-F 0 "J24" H 2450 4217 50  0000 C CNN
+F 0 "J10" H 2450 4217 50  0000 C CNN
 F 1 "Probe" H 2450 4126 50  0000 C CNN
 F 2 "Connector_PinHeader_2.54mm:PinHeader_1x02_P2.54mm_Vertical" H 2400 4000 50  0001 C CNN
@@
 AR Path="/5AC337B6/5ACBE919/5AD4C143" Ref="#PWR011"  Part="1"
 AR Path="/5AC337B6/5AD9F95A/5AD4C143" Ref="#PWR056"  Part="1"
-F 0 "#PWR056" H 2100 3850 50  0001 C CNN
+F 0 "#PWR011" H 2100 3850 50  0001 C CNN
 F 1 "GND" H 2105 3927 50  0000 C CNN
 F 2 "" H 2100 4100 50  0001 C CNN
@@
 	6000 2900 6150 2900
 $Comp
-L Connector_Specialized:Screw_Terminal_01x02 J11
+L Connector_Generic:Conn_01x02 J11
 U 1 1 5AD53BDD
 P 6750 2700
 AR Path="/5AC337B6/5ACBE919/5AD53BDD" Ref="J11"  Part="1"
 AR Path="/5AC337B6/5AD9F95A/5AD53BDD" Ref="J25"  Part="1"
-F 0 "J25" H 6829 2692 50  0000 L CNN
+F 0 "J11" H 6829 2692 50  0000 L CNN
 F 1 "Extruder Heater" H 6829 2601 50  0000 L CNN
 F 2 "PrntrBoardV1:TerminalBlock_Phoenix_PT-1,5-2-3.5-H_1x02_P3.50mm_Horizontal" H 6750 2700 50  0001 C CNN
