File: PrntrBoardV1.sch (KiCad schematic (older format))
At the start: 29 parts, among them J1 EXT 5V, J2 Bed Heater, J29 12-24V, J3 Z Probe, J30 Ext Motor Clock, J4 E0 Cool, J5 E0 Part, J6 E1 Cool, J7 E1 Part, J8 Always On Fan 1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

Commit message: Update connector components. Correct bad capacitor value.
Parts:
- C89: value 0.001uF -> 1000pf
- J1, J2, J29, J4, J5, J6, J7, J8, J9: symbol Connector_Specialized:Screw_Terminal_01x02 -> Connector_Generic:Conn_01x02
Changed lines of the file:
@@
 $EndSheet
 $Comp
-L Connector_Specialized:Screw_Terminal_01x02 J2
+L Connector_Generic:Conn_01x02 J2
 U 1 1 5AB8F2FF
 P 8100 4050
@@
 $EndSheet
 $Comp
-L Connector_Specialized:Screw_Terminal_01x02 J7
+L Connector_Generic:Conn_01x02 J7
 U 1 1 5AB92C7F
 P 9400 3350
@@
 $EndComp
 $Comp
-L Connector_Specialized:Screw_Terminal_01x02 J6
+L Connector_Generic:Conn_01x02 J6
 U 1 1 5AB92D01
 P 9400 2800
@@
 $EndComp
 $Comp
-L Connector_Specialized:Screw_Terminal_01x02 J5
+L Connector_Generic:Conn_01x02 J5
 U 1 1 5AB92D3C
 P 9400 2200
@@
 $EndComp
 $Comp
-L Connector_Specialized:Screw_Terminal_01x02 J4
+L Connector_Generic:Conn_01x02 J4
 U 1 1 5AB92D90
 P 9400 1650
@@
 	7150 5450 7150 5100
 $Comp
-L Connector_Specialized:Screw_Terminal_01x02 J8
+L Connector_Generic:Conn_01x02 J8
 U 1 1 5AC9DA10
 P 10150 1650
@@
 $EndComp
 $Comp
-L Connector_Specialized:Screw_Terminal_01x02 J9
+L Connector_Generic:Conn_01x02 J9
 U 1 1 5AC9DAC8
 P 10150 2050
@@
 Wire Wire Line
 	9900 2150 9950 2150
-Connection ~ 9950 2150
 Wire Wire Line
 	9950 2050 9850 2050
@@
 Connection ~ 4100 2900
 $Comp
-L Connector_Specialized:Screw_Terminal_01x02 J29
+L Connector_Generic:Conn_01x02 J29
 U 1 1 5ACB9063
 P 2350 900
@@
 NoConn ~ 1950 1400
 $Comp
-L Connector_Specialized:Screw_Terminal_01x02 J1
+L Connector_Generic:Conn_01x02 J1
 U 1 1 5AEDA4A7
 P 3500 1950
@@
 P 5050 1500
 F 0 "C89" H 5165 1546 50  0000 L CNN
-F 1 "0.001uF" H 5050 1400 50  0000 L CNN
+F 1 "1000pf" H 5050 1400 50  0000 L CNN
 F 2 "Capacitor_SMD:C_0603_1608Metric" H 5088 1350 50  0001 C CNN
 F 3 "~" H 5050 1500 50  0001 C CNN
