File: PrntrBoardV1.sch (KiCad schematic (older format))
At the start: 41 parts, among them J1 EXT 5V, J2 Bed Heater, J29 12-24V, J3 Z Probe, J4 E0 Cool, J5 E0 Part, J6 E1 Cool, J7 E1 Part, J8 Always On Fan 1, J9 Always On Fan 2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

Commit message: Cherry pick path names changes.
Parts:
- U2: symbol Logic_74xx:74HCT02 -> 74ls02:74HCT02
Changed lines of the file:
@@
 5V
 $Comp
-L Logic_74xx:74HCT02 U2
+L 74ls02:74HCT02 U2
 U 1 1 5AB9C30F
 P 5750 6750
@@
 $EndComp
 $Comp
-L Logic_74xx:74HCT02 U2
+L 74ls02:74HCT02 U2
 U 2 1 5AB9E04D
 P 5750 5200
@@
 $EndComp
 $Comp
-L Logic_74xx:74HCT02 U2
+L 74ls02:74HCT02 U2
 U 3 1 5AB9E0C5
 P 5750 5750
@@
 $EndComp
 $Comp
-L Logic_74xx:74HCT02 U2
+L 74ls02:74HCT02 U2
 U 4 1 5AB9E15A
 P 5750 6250
@@
 $EndComp
 $Comp
-L Logic_74xx:74HCT02 U2
+L 74ls02:74HCT02 U2
 U 5 1 5AB9E1C8
 P 7650 5600
